Commit message: Migrate rickshaw task to mjlab

File: assets/g1_dex1/g1_29dof_mode_15_with_dex1_1.urdf (robot description, URDF)
Before this commit: robot g1_29dof_mode_15, 42 links, 41 joints
Joints:
- joint left_dex1_finger_joint_1: axis 0 -1 0 -> (none); limit lower=-0.02 upper=0.0245 effort=20 velocity=0.2 -> (none); origin xyz=0 0 0 rpy=0 0 0 -> xyz=0 0.01609 0 rpy=0 0 0; type prismatic -> fixed
- joint left_dex1_finger_joint_2: axis 0 1 0 -> (none); limit lower=-0.02 upper=0.0245 effort=20 velocity=0.2 -> (none); origin xyz=0 0 0 rpy=0 0 0 -> xyz=0 -0.01609 0 rpy=0 0 0; type prismatic -> fixed
- joint right_dex1_finger_joint_1: axis 0 -1 0 -> (none); limit lower=-0.02 upper=0.0245 effort=20 velocity=0.2 -> (none); origin xyz=0 0 0 rpy=0 0 0 -> xyz=0 0.01609 0 rpy=0 0 0; type prismatic -> fixed
- joint right_dex1_finger_joint_2: axis 0 1 0 -> (none); limit lower=-0.02 upper=0.0245 effort=20 velocity=0.2 -> (none); origin xyz=0 0 0 rpy=0 0 0 -> xyz=0 -0.01609 0 rpy=0 0 0; type prismatic -> fixed

File: assets/rickshaw/rickshaw.urdf (robot description, URDF)
Before this commit: robot rickshaw, 5 links, 4 joints
Links:
- link left_wheel_link: geometry collision cylinder length=0.072548 radius=0.3; visual mesh filename=right_wheel.stl scale=0.0001 0.00008 0.00008
- link right_wheel_link: geometry collision cylinder length=0.072548 radius=0.3; visual mesh filename=left_wheel.stl scale=0.0001 0.00008 0.00008
Joints:
- joint left_tow_hitch_joint: origin xyz=1.85049373 0.235 0.18164719 rpy=0 0 0 -> xyz=1.664929 0.276 0.105747 rpy=0 0 0
- joint left_wheel_joint: origin xyz=0 0.378231 0.374999 rpy=0 0 0 -> xyz=0 0.378231 0.3 rpy=0 0 0
- joint right_tow_hitch_joint: origin xyz=1.85049373 -0.235 0.18164719 rpy=0 0 0 -> xyz=1.664929 -0.276 0.105747 rpy=0 0 0
- joint right_wheel_joint: origin xyz=0 -0.378231 0.374999 rpy=0 0 0 -> xyz=0 -0.378231 0.3 rpy=0 0 0
